File: sweetpotet_mp3.kicad_sch (KiCad schematic)
At the start: 0 parts

Commit message: Added essential components
Parts:
- added U1: STM32F072RBTx, Package_QFP:LQFP-64_10x10mm_P0.5mm, symbol MCU_ST_STM32F0:STM32F072RBTx
- added U2: AK4432VT, PCM_JLCPCB:TSSOP-16_L5.0-W4.4-P0.65-LS6.4-BL, symbol Audio_Custom:AK4432VT
- added U3, U4: NE5532DR, PCM_JLCPCB:SOIC-8_L4.9-W3.9-P1.27-LS6.0-BL, symbol PCM_JLCPCB-Analog:Op-Amp, NE5532DR
Connections:
- new net: U1.18 (VSS), U1.31 (VSS), U1.47 (VSS), U1.63 (VSS)
